File: hardware/v1/v1.kicad_sch (KiCad schematic)
At the start: 74 parts, among them J1 AUDIO IN, J10 Close for battery power, J2 MIDI OUT, J3 MIDI IN, J4 MIDI THRU, J5 OUTPUT R, J6 OUTPUT L - MONO, J7 EXP 2, J8 EXP 1, J9 Batt In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

Commit message: Replace power selection with a switch
Parts:
- removed J10: Close for battery power, Connector_PinHeader_2.54mm:PinHeader_1x02_P2.54mm_Vertical, symbol Connector:Conn_01x02_Male
- added SW2: SW_SPDT, Package_TO_SOT_THT:TO-126-3_Vertical, symbol Switch:SW_SPDT
Connections:
- net batt-: now also SW2.1 (A)
- net at J6.R: now also SW2.2 (B)
- no-connect marks 46 -> 47
Changed lines of the file:
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@@
   (no_connect (at 67.945 147.955))
   (no_connect (at 210.185 135.255))
+  (no_connect (at 453.39 87.63))
   (no_connect (at 243.205 125.095))
   (no_connect (at 101.6 74.93))
@@
     (stroke (width 0) (type default) (color 0 0 0 0))
   )
+  (wire (pts (xy 463.55 90.17) (xy 468.63 90.17))
+    (stroke (width 0) (type default) (color 0 0 0 0))
+  )
   (wire (pts (xy 43.815 137.795) (xy 43.815 139.065))
     (stroke (width 0) (type default) (color 0 0 0 0))
@@
     (stroke (width 0) (type default) (color 0 0 0 0))
   )
-  (wire (pts (xy 442.595 90.17) (xy 456.565 90.17))
-    (stroke (width 0) (type default) (color 0 0 0 0))
-  )
   (wire (pts (xy 107.95 92.71) (xy 107.95 87.63))
     (stroke (width 0) (type default) (color 0 0 0 0))
@@
     (stroke (width 0) (type default) (color 0 0 0 0))
   )
-  (wire (pts (xy 457.835 85.09) (xy 468.63 85.09))
-    (stroke (width 0) (type default) (color 0 0 0 0))
-  )
   (wire (pts (xy 396.24 45.72) (xy 396.24 46.99))
     (stroke (width 0) (type default) (color 0 0 0 0))
@@
     (stroke (width 0) (type default) (color 0 0 0 0))
   )
+  (wire (pts (xy 445.135 90.17) (xy 442.595 90.17))
+    (stroke (width 0) (type default) (color 0 0 0 0))
+  )
   (wire (pts (xy 403.86 44.45) (xy 403.86 50.8))
     (stroke (width 0) (type default) (color 0 0 0 0))
@@
     (stroke (width 0) (type default) (color 0 0 0 0))
   )
+  (wire (pts (xy 445.135 92.71) (xy 445.135 90.17))
+    (stroke (width 0) (type default) (color 0 0 0 0))
+  )
   (wire (pts (xy 191.135 127.635) (xy 191.77 127.635))
     (stroke (width 0) (type default) (color 0 0 0 0))
@@
     (stroke (width 0) (type default) (color 0 0 0 0))
   )
-  (wire (pts (xy 459.105 90.17) (xy 468.63 90.17))
-    (stroke (width 0) (type default) (color 0 0 0 0))
-  )
   (wire (pts (xy 92.71 177.8) (xy 92.71 179.705))
     (stroke (width 0) (type default) (color 0 0 0 0))
@@
     (stroke (width 0) (type default) (color 0 0 0 0))
   )
+  (wire (pts (xy 457.835 85.09) (xy 468.63 85.09))
+    (stroke (width 0) (type default) (color 0 0 0 0))
+  )
   (wire (pts (xy 59.69 33.02) (xy 72.39 33.02))
     (stroke (width 0) (type default) (color 0 0 0 0))
@@
     (stroke (width 0) (type default) (color 0 0 0 0))
   )
+  (wire (pts (xy 453.39 92.71) (xy 445.135 92.71))
+    (stroke (width 0) (type default) (color 0 0 0 0))
+  )
   (wire (pts (xy 92.71 179.705) (xy 101.6 179.705))
     (stroke (width 0) (type default) (color 0 0 0 0))
@@
     (pin "4")
   )
-  (symbol (lib_id "Connector:Conn_01x02_Male") (at 456.565 95.25 90) (unit 1)
-    (in_bom yes) (on_board yes) (fields_autoplaced)
-    (property "Reference" "J10" (id 0) (at 459.9432 93.7803 90)
-      (effects (font (size 1.27 1.27)) (justify right))
-    )
-    (property "Value" "Close for battery power" (id 1) (at 459.9432 96.3172 90)
-      (effects (font (size 1.27 1.27)) (justify right))
-    )
-    (property "Footprint" "Connector_PinHeader_2.54mm:PinHeader_1x02_P2.54mm_Vertical" (id 2) (at 456.565 95.25 0)
-      (effects (font (size 1.27 1.27)) hide)
-    )
-    (property "Datasheet" "~" (id 3) (at 456.565 95.25 0)
-      (effects (font (size 1.27 1.27)) hide)
-    )
-    (pin "1")
-    (pin "2")
-  )
   (symbol (lib_id "power:GNDA") (at 43.815 145.415 90) (unit 1)
     (in_bom yes) (on_board yes) (fields_autoplaced)
@@
     (pin "1")
   )
+  (symbol (lib_id "Switch:SW_SPDT") (at 458.47 90.17 180) (unit 1)
+    (in_bom yes) (on_board yes) (fields_autoplaced)
+    (property "Reference" "SW2" (id 0) (at 458.47 83.5492 0))
+    (property "Value" "SW_SPDT" (id 1) (at 458.47 86.0861 0))
+    (property "Footprint" "Package_TO_SOT_THT:TO-126-3_Vertical" (id 2) (at 458.47 90.17 0)
+      (effects (font (size 1.27 1.27)) hide)
+    )
+    (property "Datasheet" "~" (id 3) (at 458.47 90.17 0)
+      (effects (font (size 1.27 1.27)) hide)
+    )
+    (pin "1")
+    (pin "2")
+    (pin "3")
+  )
   (symbol (lib_id "Device:C_Polarized") (at 457.835 63.5 0) (unit 1)
     (in_bom yes) (on_board yes) (fields_autoplaced)
@@
       (reference "J9") (unit 1) (value "Batt In") (footprint "Connector_JST:JST_XH_B2B-XH-A_1x02_P2.50mm_Vertical")
     )
-    (path "/72a3182d-52e3-4382-976b-73291daa2ea7"
-      (reference "J10") (unit 1) (value "Close for battery power") (footprint "Connector_PinHeader_2.54mm:PinHeader_1x02_P2.54mm_Vertical")
-    )
     (path "/7aa8ebeb-8bea-4614-8ec6-7c790f165918"
       (reference "R1") (unit 1) (value "10") (footprint "Resistor_THT:R_Axial_DIN0207_L6.3mm_D2.5mm_P7.62mm_Horizontal")
@@
       (reference "SW1") (unit 1) (value "RotaryEncoder_Switch") (footprint "Rotary_Encoder:RotaryEncoder_Alps_EC11E-Switch_Vertical_H20mm")
     )
+    (path "/df589af9-f82b-4cf1-b85b-9090e4d02b0d"
+      (reference "SW2") (unit 1) (value "SW_SPDT") (footprint "Package_TO_SOT_THT:TO-126-3_Vertical")
+    )
     (path "/55be732d-d054-4d1b-b915-371f3d6eb5d0"
